Commit message: AR tag with fake tag

File: description/robot_core.xacro (robot description, xacro)
@@ -152,14 +152,15 @@
     </gazebo>
     <!-- AR MOUNT -->
-    <!-- <joint name="ar_mount_joint" type="fixed">
+    <joint name="ar_mount_joint" type="fixed">
         <parent link="base_link"/>
         <child link="ar_mount"/>
-        <origin xyz="${chassis_height-0.01} 0 ${chassis_length/2}"/>
+        <origin xyz="${chassis_height} 0 ${chassis_length/2}"/>
     </joint>
+    <!-- <uri>model://description/meshes/AR-tag_top.stl</uri> -->
     <link name="ar_mount">
         <visual>
             <geometry>
                 <mesh>
-                    <uri>model://meshes/AR-tag_mount_v2.STL</uri>
+                    <uri>model://description/meshes/AR-tag_top.dae</uri>
                 </mesh>
             </geometry>
@@ -169,4 +170,4 @@
     <gazebo reference="ar_mount">
         <material>Gazebo/Black</material>
-    </gazebo> -->
+    </gazebo>
 </robot>
